File: hardware/environment-sensor.kicad_pcb (KiCad board)
At the start: 2 copper layers, 80 x 75 mm, 110 parts, among them J1 J1B1211CCD, P1 POWER, P2 USB_OTG, P3 ICSP, P4 STATUS 1, P5 STATUS 2, P6 UART, P7 JTAG, P8 DS18B20, P9 PPD42, SW1 RESET, U1 LT1761-5, U2 LT1761-3.3, U3 W5500, U4 ATMEGA32U4-AU, U5 Bosch_BME280, X1 25MHz, X2 16MHz

Commit message: Finishing tweaks to revision 4
Parts:
- moved C23 3.17 mm to (158.1, 74.3)
- moved C19 1.91 mm to (184.2, 81.9)
- moved R12 1.91 mm to (184.2, 86.4)
- moved R15 0.81 mm to (182.2, 66.0)
- moved R16 0.81 mm to (182.2, 68.6)
Routing:
- net Net-(C19-Pad1): track 12.9 -> 14.5 mm
- net /Microcontroller/3V3A: track 248.1 -> 249.5 mm
- net /Network I/O/ACTLED: track 129.9 -> 128.7 mm
- net /Microcontroller/STATUS_2: track 122.2 -> 121.3 mm
- net Net-(R26-Pad2): track 87.1 -> 86.3 mm
- net /Microcontroller/STATUS_1: track 116.1 -> 115.3 mm
- net /Microcontroller/DUST_2: track 92.7 -> 91.9 mm
- net /Microcontroller/DUST_1: track 84.5 -> 83.6 mm
- net /Microcontroller/PHY_SS: track 141.4 -> 140.6 mm
- net Net-(J1-Pad9): track 3.79 -> 4.61 mm
- net /Network I/O/LINKLED: track 136.1 -> 135.4 mm, vias 4 -> 3
- net Net-(J1-Pad11): track 15.2 -> 15.8 mm
Other:
- board text added: "Rev D Sean Leavey"
- board text removed: "Sean Leavey"
