File: hardware/sensors.sch (KiCad schematic (older format))
At the start: 17 parts, among them P8 DS18B20, P9 PPD42, U5 Bosch_BME280

Commit message: Added some part numbers to the schematic
Parts:
- L5: MPN1 (none) -> 7447918; Manufacturer1 (none) -> Wurth Elektronik; SKU1 (none) -> 124-1871; Vendor1 (none) -> RS
- P8: MPN1 (none) -> 22-27-2031; Manufacturer1 (none) -> Molex; SKU1 (none) -> 483-8477; Vendor1 (none) -> RS
- P9: MPN1 (none) -> 22-27-2051; Manufacturer1 (none) -> Molex; SKU1 (none) -> 483-8499; Vendor1 (none) -> RS
- R39: Manuf1 Luna Optoelectronics -> (none); Manufacturer1 (none) -> Luna Optoelectronics; Manufacturer2 (none) -> Advanced Photonix
- U5: MPN1 (none) -> BME280; Manufacturer1 (none) -> Bosch; SKU1 (none) -> 262-BME280; Vendor1 (none) -> Mouser
Changed lines of the file:
@@
 F 2 "Sensors_LGA:Bosch_BME280_LGA-8" H 6625 1600 60  0001 C CNN
 F 3 "" H 6625 1600 60  0000 C CNN
+F 4 "Bosch" H 6625 1600 60  0001 C CNN "Manufacturer1"
+F 5 "BME280" H 6625 1600 60  0001 C CNN "MPN1"
+F 6 "Mouser" H 6625 1600 60  0001 C CNN "Vendor1"
+F 7 "262-BME280" H 6625 1600 60  0001 C CNN "SKU1"
 	1    6625 1600
 	1    0    0    -1
@@
 F 2 "Choke_SMD:Choke_SMD_1206_Standard" H 2650 1600 50  0001 C CNN
 F 3 "" H 2650 1600 50  0000 C CNN
+F 4 "Wurth Elektronik" V 2650 1600 60  0001 C CNN "Manufacturer1"
+F 5 "7447918" V 2650 1600 60  0001 C CNN "MPN1"
+F 6 "RS" V 2650 1600 60  0001 C CNN "Vendor1"
+F 7 "124-1871" V 2650 1600 60  0001 C CNN "SKU1"
 	1    2650 1600
 	0    -1   -1   0
@@
 F 2 "Connectors_Molex:Molex_KK-6410-05_05x2.54mm_Straight" H 7075 3925 50  0001 C CNN
 F 3 "" H 7075 3925 50  0000 C CNN
+F 4 "Molex" H 7075 3925 60  0001 C CNN "Manufacturer1"
+F 5 "22-27-2051" H 7075 3925 60  0001 C CNN "MPN1"
+F 6 "RS" H 7075 3925 60  0001 C CNN "Vendor1"
+F 7 "483-8499" H 7075 3925 60  0001 C CNN "SKU1"
 	1    7075 3925
 	1    0    0    -1
@@
 F 2 "Connectors_Molex:Molex_KK-6410-03_03x2.54mm_Straight" H 7075 2875 50  0001 C CNN
 F 3 "" H 7075 2875 50  0000 C CNN
+F 4 "Molex" H 7075 2875 60  0001 C CNN "Manufacturer1"
+F 5 "22-27-2031" H 7075 2875 60  0001 C CNN "MPN1"
+F 6 "RS" H 7075 2875 60  0001 C CNN "Vendor1"
+F 7 "483-8477" H 7075 2875 60  0001 C CNN "SKU1"
 	1    7075 2875
 	1    0    0    -1
@@
 F 2 "LDRs_NSL:NSL_19M51" H 7100 5425 50  0001 L BNN
 F 3 "" H 7100 5425 50  0001 L BNN
-F 4 "Luna Optoelectronics" V 7100 5425 60  0001 C CNN "Manuf1"
+F 4 "Luna Optoelectronics" V 7100 5425 60  0001 C CNN "Manufacturer1"
 F 5 "NSL-19M51" V 7100 5425 60  0001 C CNN "MPN1"
 F 6 "Digi-Key" V 7100 5425 60  0001 C CNN "Vendor1"
 F 7 "NSL-19M51-ND" V 7100 5425 60  0001 C CNN "SKU1"
-F 8 "Advanced Photonix" V 7100 5425 60  0001 C CNN "MPN2"
+F 8 "Advanced Photonix" V 7100 5425 60  0001 C CNN "Manufacturer2"
 F 9 "NSL 19M51" V 7100 5425 60  0001 C CNN "MPN2"
 F 10 "Farnell" V 7100 5425 60  0001 C CNN "Vendor2"
